Commit message: KYS CAD add mapping

File: 2_wheel_robot/model/wheel_robot.urdf (robot description, URDF)
Before this commit: robot wheel_robot, 5 links, 4 joints
Links:
- added link imu_link, mass 0.05; collision box size=0.04 0.03 0.01; visual box size=0.04 0.03 0.01
Joints:
- added joint imu_joint: type fixed, parent base_link, child imu_link, origin xyz=-0.08 0 0.055 rpy=0 0 0
- joint left_wheel_joint: limit effort=10.0 velocity=20.0 -> effort=20.0 velocity=20.0
- joint right_wheel_joint: limit effort=10.0 velocity=20.0 -> effort=20.0 velocity=20.0
